File: power_rev2.kicad_sch (KiCad schematic)
At the start: 27 parts, among them J1 Conn_02x03_Odd_Even, J2 Conn_01x02_Pin, J4 Conn_01x04_Pin, U2 ESP32-S3-WROOM-1, U4 MCP1825S

Commit message: added name: noah
Other:
- note added: "Noah"
Changed lines of the file:
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@@
+		)
+	)
+	(text "Noah"
+		(exclude_from_sim no)
+		(at 240.03 133.858 0)
+		(effects
+			(font
+				(size 1.27 1.27)
+			)
 		)
 	)

Commit message: Added my name
Other:
- note added: "William"
Changed lines of the file:
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@@
+		)
+	)
+	(text "William\n"
+		(exclude_from_sim no)
+		(at 258.826 144.526 0)
+		(effects
+			(font
+				(size 1.27 1.27)
+			)
 		)
 	)

Commit message: Added name
Other:
- note added: "Vic"
Changed lines of the file:
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@@
+		)
+	)
+	(text "Vic"
+		(exclude_from_sim no)
+		(at 238.252 145.034 0)
+		(effects
+			(font
+				(size 1.27 1.27)
+			)
 		)
 	)

Commit message: Added name
Other:
- note added: "Francis"
Changed lines of the file:
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@@
+		)
+	)
+	(text "Francis"
+		(exclude_from_sim no)
+		(at 250.698 152.4 0)
+		(effects
+			(font
+				(size 1.27 1.27)
+			)
 		)
 	)

Commit message: I added my name
Other:
- note added: "Eason"
Changed lines of the file:
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@@
+		)
+	)
+	(text "Eason"
+		(exclude_from_sim no)
+		(at 256.286 132.842 0)
+		(effects
+			(font
+				(size 1.27 1.27)
+			)
 		)
 	)

Commit message: I added my name
Other:
- note added: "Maggie"
Changed lines of the file:
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@@
+		)
+	)
+	(text "Maggie"
+		(exclude_from_sim no)
+		(at 247.904 126.746 0)
+		(effects
+			(font
+				(size 1.27 1.27)
+			)
 		)
 	)
