File: power_rev2.kicad_sch (KiCad schematic)
At the start: 27 parts, among them J1 Conn_02x03_Odd_Even, J2 Conn_01x02_Pin, J4 Conn_01x04_Pin, U2 ESP32-S3-WROOM-1, U4 MCP1825S

Commit message: added name shawn
Other:
- note added: "shawn"
Changed lines of the file:
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@@
+		)
+	)
+	(text "shawn"
+		(exclude_from_sim no)
+		(at 230.632 154.686 0)
+		(effects
+			(font
+				(size 1.27 1.27)
+			)
 		)
 	)
