File: Crank power meter.kicad_sch (KiCad schematic)
At the start: 26 parts, among them J4 Conn_01x04_Pin, Q1 PNP, U1 ESP32-S3-MINI-1, U2 MCP1825S, U3 HX711

Commit message: added ESP prog
Parts:
- added J1: Conn_02x03_Odd_Even, Connector_IDC:IDC-Header_2x03_P2.54mm_Vertical, symbol Connector_Generic:Conn_02x03_Odd_Even
Connections:
- net +3.3V: now also J1.4 (Pin_4)
- net +3V3: now also J1.2 (Pin_2)
Other:
- note added: "Programming (ESP PROG)"
- note removed: "2"
- note removed: "HPVDT Crank Power Meter"
